Commit message: update max velocity for kr6r900-2 from manual for rated payload 3k

File: kuka_kr6_support/urdf/kr6r900_2_macro.xacro (robot description, xacro)
@@ -137,5 +137,5 @@
       <child link="${prefix}link_4"/>
       <axis xyz="-1 0 0"/>
-      <limit effort="0" lower="${-DEG2RAD * 185}" upper="${DEG2RAD * 185}" velocity="${DEG2RAD * 381}"/>
+      <limit effort="0" lower="${-DEG2RAD * 185}" upper="${DEG2RAD * 185}" velocity="${DEG2RAD * 450}"/>
     </joint>
     <joint name="${prefix}joint_a5" type="revolute">
@@ -144,5 +144,5 @@
       <child link="${prefix}link_5"/>
       <axis xyz="0 1 0"/>
-      <limit effort="0" lower="${-DEG2RAD * 120}" upper="${DEG2RAD * 120}" velocity="${DEG2RAD * 388}"/>
+      <limit effort="0" lower="${-DEG2RAD * 120}" upper="${DEG2RAD * 120}" velocity="${DEG2RAD * 450}"/>
     </joint>
     <joint name="${prefix}joint_a6" type="revolute">
@@ -151,5 +151,5 @@
       <child link="${prefix}link_6"/>
       <axis xyz="-1 0 0"/>
-      <limit effort="0" lower="${-DEG2RAD * 350}" upper="${DEG2RAD * 350}" velocity="${DEG2RAD * 615}"/>
+      <limit effort="0" lower="${-DEG2RAD * 350}" upper="${DEG2RAD * 350}" velocity="${DEG2RAD * 540}"/>
     </joint>
     <joint name="${prefix}joint_a6-tool0" type="fixed">

Commit message: kr6r900-2: use identical visual&coll from kr10r900-2

File: kuka_kr6_support/urdf/kr6r900_2_macro.xacro (robot description, xacro)
@@ -8,12 +8,12 @@
         <origin xyz="0 0 0" rpy="0 0 0"/>
         <geometry>
-          <mesh filename="package://kuka_kr6_support/meshes/kr6_agilus/visual/base_link.dae" />
+          <mesh filename="package://kuka_kr10_support/meshes/kr10r900_2/visual/base_link.stl" />
         </geometry>
-        <xacro:material_kuka_pedestal />
+        <xacro:material_kuka_ral_gray_aluminium />
       </visual>
       <collision>
         <origin xyz="0 0 0" rpy="0 0 0"/>
         <geometry>
-          <mesh filename="package://kuka_kr6_support/meshes/kr6_agilus/collision/base_link.stl" />
+          <mesh filename="package://kuka_kr10_support/meshes/kr10r900_2/collision/base_link.stl" />
         </geometry>
       </collision>
@@ -23,12 +23,12 @@
         <origin xyz="0 0 0" rpy="0 0 0"/>
         <geometry>
-          <mesh filename="package://kuka_kr6_support/meshes/kr6_agilus/visual/link_1.dae" />
+          <mesh filename="package://kuka_kr10_support/meshes/kr10r900_2/visual/link_1.stl" />
         </geometry>
-        <xacro:material_kuka_orange />
+        <xacro:material_kuka_ral_traffic_white />
       </visual>
       <collision>
         <origin xyz="0 0 0" rpy="0 0 0"/>
         <geometry>
-          <mesh filename="package://kuka_kr6_support/meshes/kr6_agilus/collision/link_1.stl" />
+          <mesh filename="package://kuka_kr10_support/meshes/kr10r900_2/collision/link_1.stl" />
         </geometry>
       </collision>
@@ -38,12 +38,12 @@
         <origin xyz="0 0 0" rpy="0 0 0"/>
         <geometry>
-          <mesh filename="package://kuka_kr6_support/meshes/kr6r900_2/visual/link_2.dae"/>
+          <mesh filename="package://kuka_kr10_support/meshes/kr10r900_2/visual/link_2.stl"/>
         </geometry>
-        <xacro:material_kuka_orange />
+        <xacro:material_kuka_ral_traffic_white />
       </visual>
       <collision>
         <origin xyz="0 0 0" rpy="0 0 0"/>
         <geometry>
-          <mesh filename="package://kuka_kr6_support/meshes/kr6r900_2/collision/link_2.stl" />
+          <mesh filename="package://kuka_kr10_support/meshes/kr10r900_2/collision/link_2.stl" />
         </geometry>
       </collision>
@@ -53,12 +53,12 @@
         <origin xyz="0 0 0" rpy="0 0 0"/>
         <geometry>
-          <mesh filename="package://kuka_kr6_support/meshes/kr6_agilus/visual/link_3.dae" />
+          <mesh filename="package://kuka_kr10_support/meshes/kr10r900_2/visual/link_3.stl" />
         </geometry>
-        <xacro:material_kuka_orange />
+        <xacro:material_kuka_ral_traffic_white />
       </visual>
       <collision>
         <origin xyz="0 0 0" rpy="0 0 0"/>
         <geometry>
-          <mesh filename="package://kuka_kr6_support/meshes/kr6_agilus/collision/link_3.stl" />
+          <mesh filename="package://kuka_kr10_support/meshes/kr10r900_2/collision/link_3.stl" />
         </geometry>
       </collision>
@@ -68,12 +68,12 @@
         <origin xyz="0 0 0" rpy="0 0 0"/>
         <geometry>
-          <mesh filename="package://kuka_kr6_support/meshes/kr6r900_2/visual/link_4.dae" />
+          <mesh filename="package://kuka_kr10_support/meshes/kr10r900_2/visual/link_4.stl" />
         </geometry>
-        <xacro:material_kuka_orange />
+        <xacro:material_kuka_ral_traffic_white />
       </visual>
       <collision>
         <origin xyz="0 0 0" rpy="0 0 0"/>
         <geometry>
-          <mesh filename="package://kuka_kr6_support/meshes/kr6r900_2/collision/link_4.stl" />
+          <mesh filename="package://kuka_kr10_support/meshes/kr10r900_2/collision/link_4.stl" />
         </geometry>
       </collision>
@@ -83,12 +83,12 @@
         <origin xyz="0 0 0" rpy="0 0 0"/>
         <geometry>
-          <mesh filename="package://kuka_kr6_support/meshes/kr6_agilus/visual/link_5.dae" />
+          <mesh filename="package://kuka_kr10_support/meshes/kr10r900_2/visual/link_5.stl" />
         </geometry>
-        <xacro:material_kuka_orange />
+        <xacro:material_kuka_ral_traffic_white />
       </visual>
       <collision>
         <origin xyz="0 0 0" rpy="0 0 0"/>
         <geometry>
-          <mesh filename="package://kuka_kr6_support/meshes/kr6_agilus/collision/link_5.stl" />
+          <mesh filename="package://kuka_kr10_support/meshes/kr10r900_2/collision/link_5.stl" />
         </geometry>
       </collision>
@@ -98,12 +98,12 @@
         <origin xyz="0 0 0" rpy="0 0 0"/>
         <geometry>
-          <mesh filename="package://kuka_kr6_support/meshes/kr6_agilus/visual/link_6.dae" />
+          <mesh filename="package://kuka_kr10_support/meshes/kr10r900_2/visual/link_6.stl" />
         </geometry>
-        <xacro:material_kuka_pedestal />
+        <xacro:material_kuka_black />
       </visual>
       <collision>
         <origin xyz="0 0 0" rpy="0 0 0"/>
         <geometry>
-          <mesh filename="package://kuka_kr6_support/meshes/kr6_agilus/collision/link_6.stl" />
+          <mesh filename="package://kuka_kr10_support/meshes/kr10r900_2/collision/link_6.stl" />
         </geometry>
       </collision>

Commit message: use radians function instead of macro

File: kuka_kr6_support/urdf/kr6r900_2_macro.xacro (robot description, xacro)
@@ -116,5 +116,5 @@
       <child link="${prefix}link_1"/>
       <axis xyz="0 0 -1"/>
-      <limit effort="0" lower="${-DEG2RAD * 170}" upper="${DEG2RAD * 170}" velocity="${DEG2RAD * 360}"/>
+      <limit effort="0" lower="${radians(-170)}" upper="${radians(170)}" velocity="${radians(360)}"/>
     </joint>
     <joint name="${prefix}joint_a2" type="revolute">
@@ -123,5 +123,5 @@
       <child link="${prefix}link_2"/>
       <axis xyz="0 1 0"/>
-      <limit effort="0" lower="${-DEG2RAD * 190}" upper="${DEG2RAD * 45}" velocity="${DEG2RAD * 300}"/>
+      <limit effort="0" lower="${radians(-190)}" upper="${radians(45)}" velocity="${radians(300)}"/>
     </joint>
     <joint name="${prefix}joint_a3" type="revolute">
@@ -130,5 +130,5 @@
       <child link="${prefix}link_3"/>
       <axis xyz="0 1 0"/>
-      <limit effort="0" lower="${-DEG2RAD * 120}" upper="${DEG2RAD * 156}" velocity="${DEG2RAD * 360}"/>
+      <limit effort="0" lower="${radians(-120)}" upper="${radians(156)}" velocity="${radians(360)}"/>
     </joint>
     <joint name="${prefix}joint_a4" type="revolute">
@@ -137,5 +137,5 @@
       <child link="${prefix}link_4"/>
       <axis xyz="-1 0 0"/>
-      <limit effort="0" lower="${-DEG2RAD * 185}" upper="${DEG2RAD * 185}" velocity="${DEG2RAD * 450}"/>
+      <limit effort="0" lower="${radians(-185)}" upper="${radians(185)}" velocity="${radians(450)}"/>
     </joint>
     <joint name="${prefix}joint_a5" type="revolute">
@@ -144,5 +144,5 @@
       <child link="${prefix}link_5"/>
       <axis xyz="0 1 0"/>
-      <limit effort="0" lower="${-DEG2RAD * 120}" upper="${DEG2RAD * 120}" velocity="${DEG2RAD * 450}"/>
+      <limit effort="0" lower="${radians(-120)}" upper="${radians(120)}" velocity="${radians(450)}"/>
     </joint>
     <joint name="${prefix}joint_a6" type="revolute">
@@ -151,10 +151,10 @@
       <child link="${prefix}link_6"/>
       <axis xyz="-1 0 0"/>
-      <limit effort="0" lower="${-DEG2RAD * 350}" upper="${DEG2RAD * 350}" velocity="${DEG2RAD * 540}"/>
+      <limit effort="0" lower="${radians(-350)}" upper="${radians(350)}" velocity="${radians(540)}"/>
     </joint>
     <joint name="${prefix}joint_a6-tool0" type="fixed">
       <parent link="${prefix}link_6"/>
       <child link="${prefix}tool0"/>
-      <origin xyz="0 0 0" rpy="0 ${DEG2RAD * 90} 0"/>
+      <origin xyz="0 0 0" rpy="0 ${radians(90)} 0"/>
     </joint>
     <!-- ROS base_link to KUKA $ROBROOT coordinate system transform -->
