Commit message: Configuring for use on kr60 Added t1 tag for kr60 which sets the velocity limit for all joints to 30 deg Got the simulator working without ros though.

File: kuka_kr60_support/urdf/kr60.ros2_control.xacro (robot description, xacro)
@@ -1,11 +1,11 @@
 <?xml version="1.0"?>
 <robot xmlns:xacro="http://www.ros.org/wiki/xacro">
-    <xacro:macro name="kr_60_position" params="name robot_ip robot_port hardware:=false linear_rail:=false">
+    <xacro:macro name="kr_60_position" params="name listen_ip listen_port hardware:=false linear_rail:=false">
         <ros2_control name="${name}" type="system">
             <hardware>
                 <xacro:if value="${hardware}">
                     <plugin>kuka_rsi_hw_interface/KukaHardwareInterface</plugin>
-                    <param name="robot_ip">${robot_ip}</param>
-                    <param name="robot_port">${robot_port}</param>
+                    <param name="listen_ip">${listen_ip}</param>
+                    <param name="listen_port">${listen_port}</param>
                 </xacro:if>
                 <xacro:unless value="${hardware}">

File: kuka_kr60_support/urdf/kr60ha_macro.xacro (robot description, xacro)
@@ -1,5 +1,5 @@
 <?xml version="1.0"?>
 <robot xmlns:xacro="http://wiki.ros.org/xacro">
-  <xacro:macro name="kuka_kr60ha" params="prefix">
+  <xacro:macro name="kuka_kr60ha" params="prefix t1">
     <xacro:include filename="$(find kuka_resources)/urdf/common_materials.xacro"/>
     <!-- LINKS -->
@@ -154,5 +154,10 @@
       <child link="${prefix}link_1"/>
       <axis xyz="0 0 -1"/>
-      <limit effort="0" lower="${-radians(185)}" upper="${radians(185)}" velocity="${radians(128)}"/>
+      <xacro:if value="${t1}">
+        <limit effort="0" lower="${-radians(185)}" upper="${radians(185)}" velocity="${radians(30)}"/>
+      </xacro:if>
+      <xacro:unless value="${t1}">
+        <limit effort="0" lower="${-radians(185)}" upper="${radians(185)}" velocity="${radians(128)}"/>
+      </xacro:unless>
     </joint>
     <!-- joint 2 (A2) -->
@@ -162,5 +167,10 @@
       <child link="${prefix}link_2"/>
       <axis xyz="0 1 0"/>
-      <limit effort="0" lower="${-radians(135)}" upper="${radians(35)}" velocity="${radians(102)}"/>
+      <xacro:if value="${t1}">
+        <limit effort="0" lower="${-radians(185)}" upper="${radians(185)}" velocity="${radians(30)}"/>
+      </xacro:if>
+      <xacro:unless value="${t1}">
+        <limit effort="0" lower="${-radians(185)}" upper="${radians(185)}" velocity="${radians(102)}"/>
+      </xacro:unless>
     </joint>
     <!-- joint 3 (A3) -->
@@ -170,5 +180,10 @@
       <child link="${prefix}link_3"/>
       <axis xyz="0 1 0"/>
-      <limit effort="0" lower="${-radians(120)}" upper="${radians(158)}" velocity="${radians(128)}"/>
+      <xacro:if value="${t1}">
+        <limit effort="0" lower="${-radians(185)}" upper="${radians(185)}" velocity="${radians(30)}"/>
+      </xacro:if>
+      <xacro:unless value="${t1}">
+        <limit effort="0" lower="${-radians(185)}" upper="${radians(185)}" velocity="${radians(128)}"/>
+      </xacro:unless>
     </joint>
     <!-- joint 4 (A4) -->
@@ -178,5 +193,10 @@
       <child link="${prefix}link_4"/>
       <axis xyz="-1 0 0"/>
-      <limit effort="0" lower="${-radians(350)}" upper="${radians(350)}" velocity="${radians(260)}"/>
+      <xacro:if value="${t1}">
+        <limit effort="0" lower="${-radians(185)}" upper="${radians(185)}" velocity="${radians(30)}"/>
+      </xacro:if>
+      <xacro:unless value="${t1}">
+        <limit effort="0" lower="${-radians(185)}" upper="${radians(185)}" velocity="${radians(260)}"/>
+      </xacro:unless>
     </joint>
     <!-- joint 5 (A5) -->
@@ -186,5 +206,10 @@
       <child link="${prefix}link_5"/>
       <axis xyz="0 1 0"/>
-      <limit effort="0" lower="${-radians(119)}" upper="${radians(119)}" velocity="${radians(245)}"/>
+      <xacro:if value="${t1}">
+        <limit effort="0" lower="${-radians(185)}" upper="${radians(185)}" velocity="${radians(30)}"/>
+      </xacro:if>
+      <xacro:unless value="${t1}">
+        <limit effort="0" lower="${-radians(185)}" upper="${radians(185)}" velocity="${radians(245)}"/>
+      </xacro:unless>
     </joint>
     <!-- joint 6 (A6) -->
@@ -194,5 +219,10 @@
       <child link="${prefix}link_6"/>
       <axis xyz="-1 0 0"/>
-      <limit effort="0" lower="${-radians(350)}" upper="${radians(350)}" velocity="${radians(322)}"/>
+      <xacro:if value="${t1}">
+        <limit effort="0" lower="${-radians(185)}" upper="${radians(185)}" velocity="${radians(30)}"/>
+      </xacro:if>
+      <xacro:unless value="${t1}">
+        <limit effort="0" lower="${-radians(185)}" upper="${radians(185)}" velocity="${radians(322)}"/>
+      </xacro:unless>
     </joint>
     <!-- tool frame - fixed frame -->
